File: PCB/_autosave-thermoelectric-tube.kicad_pcb (KiCad board)
At the start: 2 copper layers, 142.2 x 91.4 mm, 32 parts, among them J1 Barrel_Jack, M1 Fan, M2 Fan, Q1 2N3904, Q2 IRF9630, Q3 IRF630, Q4 2N3904, Q5 IRF9630, Q6 IRF630, U1 AD595AQ

Commit message: revB
Other:
- rule pad_to_mask_clearance: 0.051 -> 0
