File: PCB/thermoelectric-tube.sch (KiCad schematic (older format))
At the start: 23 parts, among them J1 Barrel_Jack, Q1 2N3904, Q2 IRF9630, Q3 IRF630, Q4 2N3904, Q5 IRF9630, Q6 IRF630, U1 AD595AQ

Commit message: fans
Parts:
- added M? (x2): Fan, symbol Motor:Fan
Connections:
- net +12V: now also M?.1 (+), M?.1 (+)
- net GND: now also M?.2 (-), M?.2 (-)
Changed lines of the file:
@@
 EESchema Schematic File Version 4
-LIBS:thermoelectric-tube-cache
 EELAYER 30 0
 EELAYER END
@@
 Sheet 1 1
 Title "Thermoelectric Tube"
-Date "2019-08-14"
-Rev "1.1.0"
+Date "2021-07-26"
+Rev "B"
 Comp "UW-Madison"
 Comment1 "Department of Chemistry"
-Comment2 "Blaise Thompson"
-Comment3 "bthompson@chem.wisc.edu"
-Comment4 ""
+Comment2 "Instrument Shop"
+Comment3 "Blaise Thompson"
+Comment4 "blaise.thompson@wisc.edu"
 $EndDescr
 $Comp
@@
 Wire Wire Line
 	7350 4050 7350 4600
+$Comp
+L Motor:Fan M?
+U 1 1 60FF5EEF
+P 1500 5800
+F 0 "M?" H 1658 5896 50  0000 L CNN
+F 1 "Fan" H 1658 5805 50  0000 L CNN
+F 2 "" H 1500 5810 50  0001 C CNN
+F 3 "~" H 1500 5810 50  0001 C CNN
+	1    1500 5800
+	1    0    0    -1
+$EndComp
+$Comp
+L Motor:Fan M?
+U 1 1 60FF71DB
+P 2500 5800
+F 0 "M?" H 2658 5896 50  0000 L CNN
+F 1 "Fan" H 2658 5805 50  0000 L CNN
+F 2 "" H 2500 5810 50  0001 C CNN
+F 3 "~" H 2500 5810 50  0001 C CNN
+	1    2500 5800
+	1    0    0    -1
+$EndComp
+$Comp
+L power:GND #PWR?
+U 1 1 60FF7A6C
+P 1500 6000
+F 0 "#PWR?" H 1500 5750 50  0001 C CNN
+F 1 "GND" H 1505 5827 50  0000 C CNN
+F 2 "" H 1500 6000 50  0001 C CNN
+F 3 "" H 1500 6000 50  0001 C CNN
+	1    1500 6000
+	1    0    0    -1
+$EndComp
+$Comp
+L power:GND #PWR?
+U 1 1 60FF7D4D
+P 2500 6000
+F 0 "#PWR?" H 2500 5750 50  0001 C CNN
+F 1 "GND" H 2505 5827 50  0000 C CNN
+F 2 "" H 2500 6000 50  0001 C CNN
+F 3 "" H 2500 6000 50  0001 C CNN
+	1    2500 6000
+	1    0    0    -1
+$EndComp
+$Comp
+L power:+12V #PWR?
+U 1 1 60FF83E8
+P 1500 5500
+F 0 "#PWR?" H 1500 5350 50  0001 C CNN
+F 1 "+12V" H 1515 5673 50  0000 C CNN
+F 2 "" H 1500 5500 50  0001 C CNN
+F 3 "" H 1500 5500 50  0001 C CNN
+	1    1500 5500
+	1    0    0    -1
+$EndComp
+$Comp
+L power:+12V #PWR?
+U 1 1 60FF8708
+P 2500 5500
+F 0 "#PWR?" H 2500 5350 50  0001 C CNN
+F 1 "+12V" H 2515 5673 50  0000 C CNN
+F 2 "" H 2500 5500 50  0001 C CNN
+F 3 "" H 2500 5500 50  0001 C CNN
+	1    2500 5500
+	1    0    0    -1
+$EndComp
 $EndSCHEMATC

Commit message: revB
Parts:
- M1, M2: renamed from M?; footprint (none) -> footprints:F17HA-05HC
- TC1: footprint Connector_Wire:SolderWirePad_1x02_P5.08mm_Drill1.5mm -> Connector_Molex:Molex_Mini-Fit_Jr_5566-02A_2x01_P4.20mm_Vertical
Changed lines of the file:
@@
 F 0 "TC1" V 1527 756 50  0000 R CNN
 F 1 "Thermocouple" V 1618 756 50  0000 R CNN
-F 2 "Connector_Wire:SolderWirePad_1x02_P5.08mm_Drill1.5mm" H 1025 950 50  0001 C CNN
+F 2 "Connector_Molex:Molex_Mini-Fit_Jr_5566-02A_2x01_P4.20mm_Vertical" H 1025 950 50  0001 C CNN
 F 3 "~" H 1025 950 50  0001 C CNN
 	1    1600 900
@@
 	7350 4050 7350 4600
 $Comp
-L Motor:Fan M?
+L Motor:Fan M1
 U 1 1 60FF5EEF
 P 1500 5800
-F 0 "M?" H 1658 5896 50  0000 L CNN
+F 0 "M1" H 1658 5896 50  0000 L CNN
 F 1 "Fan" H 1658 5805 50  0000 L CNN
-F 2 "" H 1500 5810 50  0001 C CNN
+F 2 "footprints:F17HA-05HC" H 1500 5810 50  0001 C CNN
 F 3 "~" H 1500 5810 50  0001 C CNN
 	1    1500 5800
@@
 $EndComp
 $Comp
-L Motor:Fan M?
+L Motor:Fan M2
 U 1 1 60FF71DB
 P 2500 5800
-F 0 "M?" H 2658 5896 50  0000 L CNN
+F 0 "M2" H 2658 5896 50  0000 L CNN
 F 1 "Fan" H 2658 5805 50  0000 L CNN
-F 2 "" H 2500 5810 50  0001 C CNN
+F 2 "footprints:F17HA-05HC" H 2500 5810 50  0001 C CNN
 F 3 "~" H 2500 5810 50  0001 C CNN
 	1    2500 5800
@@
 $EndComp
 $Comp
-L power:GND #PWR?
+L power:GND #PWR0119
 U 1 1 60FF7A6C
 P 1500 6000
-F 0 "#PWR?" H 1500 5750 50  0001 C CNN
+F 0 "#PWR0119" H 1500 5750 50  0001 C CNN
 F 1 "GND" H 1505 5827 50  0000 C CNN
 F 2 "" H 1500 6000 50  0001 C CNN
@@
 $EndComp
 $Comp
-L power:GND #PWR?
+L power:GND #PWR0120
 U 1 1 60FF7D4D
 P 2500 6000
-F 0 "#PWR?" H 2500 5750 50  0001 C CNN
+F 0 "#PWR0120" H 2500 5750 50  0001 C CNN
 F 1 "GND" H 2505 5827 50  0000 C CNN
 F 2 "" H 2500 6000 50  0001 C CNN
@@
 $EndComp
 $Comp
-L power:+12V #PWR?
+L power:+12V #PWR0121
 U 1 1 60FF83E8
 P 1500 5500
-F 0 "#PWR?" H 1500 5350 50  0001 C CNN
+F 0 "#PWR0121" H 1500 5350 50  0001 C CNN
 F 1 "+12V" H 1515 5673 50  0000 C CNN
 F 2 "" H 1500 5500 50  0001 C CNN
@@
 $EndComp
 $Comp
-L power:+12V #PWR?
+L power:+12V #PWR0122
 U 1 1 60FF8708
 P 2500 5500
-F 0 "#PWR?" H 2500 5350 50  0001 C CNN
+F 0 "#PWR0122" H 2500 5350 50  0001 C CNN
 F 1 "+12V" H 2515 5673 50  0000 C CNN
 F 2 "" H 2500 5500 50  0001 C CNN
