File: pcb/thermoelectric-tube.kicad_pcb (KiCad board)
At the start: 2 copper layers, 142.2 x 91.4 mm, 32 parts, among them J1 Barrel_Jack, M1 Fan, M2 Fan, Q1 2N3904, Q2 IRF9630, Q3 IRF630, Q4 2N3904, Q5 IRF9630, Q6 IRF630, U1 AD595AQ

Commit message: catchup
Parts:
- removed the REF** at (129.5, 116.8)
- removed TC1: Thermocouple, Connector_Wire:SolderWire-2sqmm_1x02_P7.8mm_D2mm_OD3.9mm
- removed XA1: Arduino_Micro_Socket, Arduino:Arduino_Micro_Socket
- added C3: 22u, Capacitor_THT:C_Radial_D6.3mm_H5.0mm_P2.50mm, F.Cu at (71.1, 81.3)
- added C4: 20p, Capacitor_THT:C_Radial_D6.3mm_H5.0mm_P2.50mm, F.Cu at (66.0, 127.0)
- added C5: 20p, Capacitor_THT:C_Radial_D6.3mm_H5.0mm_P2.50mm, F.Cu at (76.2, 127.0)
- added D4: LED, LED_THT:LED_D5.0mm, F.Cu at (94.0, 127.0)
- added D5: LED, LED_THT:LED_D5.0mm, F.Cu at (104.1, 127.0)
- added D6: LED, LED_THT:LED_D5.0mm, F.Cu at (114.3, 127.0)
- added D7: LED, LED_THT:LED_D5.0mm, F.Cu at (124.5, 127.0)
- added D8: LED, LED_THT:LED_D5.0mm, F.Cu at (134.6, 127.0)
- added PS1: VXO7805-500-M, footprints:CONV_VXO7805-500-M, F.Cu at (55.9, 76.2)
- added R10: 1M, Resistor_THT:R_Axial_DIN0207_L6.3mm_D2.5mm_P7.62mm_Horizontal, F.Cu at (67.3, 111.8)
- added R11: 1k, Resistor_THT:R_Axial_DIN0207_L6.3mm_D2.5mm_P7.62mm_Horizontal, F.Cu at (114.3, 113.0)
- added R12: 1k, Resistor_THT:R_Axial_DIN0207_L6.3mm_D2.5mm_P7.62mm_Horizontal, F.Cu at (124.5, 113.0)
- added R13: 1k, Resistor_THT:R_Axial_DIN0207_L6.3mm_D2.5mm_P7.62mm_Horizontal, F.Cu at (134.6, 113.0)
- added R8: 1k, Resistor_THT:R_Axial_DIN0207_L6.3mm_D2.5mm_P7.62mm_Horizontal, F.Cu at (94.0, 113.0)
- added R9: 1k, Resistor_THT:R_Axial_DIN0207_L6.3mm_D2.5mm_P7.62mm_Horizontal, F.Cu at (104.1, 113.0)
- added REF**: OSHW-Logo2_14.6x12mm_SilkScreen, Symbol:OSHW-Logo2_14.6x12mm_SilkScreen, B.Cu at (83.8, 58.4)
- added SW1: SW_Push, footprints:PTS636, F.Cu at (142.2, 124.5)
- added SW2: SW_Push, footprints:PTS636, F.Cu at (86.4, 124.5)
- added TP1: TestPoint, TestPoint:TestPoint_Loop_D2.60mm_Drill1.6mm_Beaded, F.Cu at (106.7, 48.3)
- added TP2: TestPoint, TestPoint:TestPoint_Loop_D2.60mm_Drill1.6mm_Beaded, F.Cu at (114.3, 48.3)
- added TP3: TestPoint, TestPoint:TestPoint_Loop_D2.60mm_Drill1.6mm_Beaded, F.Cu at (137.2, 48.3)
- added TP4: TestPoint, TestPoint:TestPoint_Loop_D2.60mm_Drill1.6mm_Beaded, F.Cu at (144.8, 48.3)
- added TP5: TestPoint, TestPoint:TestPoint_Loop_D2.60mm_Drill1.6mm_Beaded, F.Cu at (99.1, 48.3)
- added Y1: 16MHz, Crystal:Crystal_HC49-U_Vertical, F.Cu at (73.7, 119.4)
- C1: value CP1 -> 100u
- C2: value 100n -> 10u
- R1, R2, R7: value 10k -> 1k
- R6: value R_US -> 10k
- U1: value AD595AQ -> ATmega328-P; footprint Package_DIP:DIP-14_W7.62mm_Socket_LongPads -> Package_DIP:DIP-28_W7.62mm
- moved C2 38.1 mm to (61.0, 61.0)
- moved R1 29.0 mm to (64.8, 91.4), turned to 180 degrees
- moved U1 27.2 mm to (49.5, 105.4), turned to 90 degrees
- moved D1 18.0 mm to (48.3, 91.4), turned to 0 degrees
- moved C1 11.4 mm to (71.1, 66.0)
Connections:
- C2 pad 1: GND -> +12V
- C2 pad 2: +5V -> GND
- R1 pad 1: Net-(D1-Pad2) -> +5V
- R1 pad 2: +12V -> Net-(D1-Pad2)
- R2 pad 2: Net-(R2-Pad2) -> HEAT
- R3 pad 1: Net-(R2-Pad2) -> HEAT
- R6 pad 2: Net-(R6-Pad2) -> COOL
- R7 pad 2: Net-(R6-Pad2) -> COOL
- U1 pad 1: GND -> unconnected-(U1-Pad1)
- U1 pad 10: (no net) -> Net-(C5-Pad2)
- U1 pad 11: +5V -> Net-(R11-Pad1)
- U1 pad 12: (no net) -> Net-(R9-Pad1)
- U1 pad 13: GND -> Net-(R8-Pad1)
- U1 pad 14: Net-(TC1-Pad2) -> unconnected-(U1-Pad14)
- U1 pad 2: (no net) -> Net-(SW1-Pad1)
- U1 pad 3: (no net) -> Net-(SW2-Pad1)
- U1 pad 4: GND -> unconnected-(U1-Pad4)
- U1 pad 5: (no net) -> Net-(R13-Pad1)
- U1 pad 6: (no net) -> Net-(R12-Pad1)
- U1 pad 7: GND -> +5V
- U1 pad 8: Net-(U1-Pad8) -> GND
- U1 pad 9: Net-(U1-Pad8) -> Net-(C4-Pad1)
Routing:
- net Net-(SW1-Pad1): track 0.00 -> 114.0 mm
- net Net-(R6-Pad2): track 108.3 -> 0.00 mm
- net Net-(R2-Pad2): track 108.3 -> 0.00 mm
- net HEAT: track 0.00 -> 94.0 mm
- net COOL: track 0.00 -> 93.0 mm
- net Net-(R13-Pad1): track 0.00 -> 84.2 mm
- net Net-(R12-Pad1): track 0.00 -> 70.0 mm
- net Net-(U1-Pad8): track 54.0 -> 0.00 mm
- net +5V: track 68.1 -> 118.8 mm
- net Net-(R11-Pad1): track 0.00 -> 44.0 mm
- net Net-(SW2-Pad1): track 0.00 -> 41.3 mm
- net +12V: track 33.6 -> 74.1 mm
- net Net-(R9-Pad1): track 0.00 -> 35.2 mm
- net Net-(PE1-Pad1): track 44.0 -> 72.7 mm
- net Net-(C4-Pad1): track 0.00 -> 24.3 mm
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Other:
- net class Default removed
- rule pad_to_mask_clearance: 0.051 -> 0
- board text added: "REVISION C JULY 2022"
- board text removed: "POWER"
- board text removed: "REVISION B JULY 2021"
