File: pcb/thermoelectric-tube.sch (KiCad schematic (older format))
At the start: 25 parts, among them J1 Barrel_Jack, M1 Fan, M2 Fan, Q1 2N3904, Q2 IRF9630, Q3 IRF630, Q4 2N3904, Q5 IRF9630, Q6 IRF630, U1 AD595AQ

Commit message: catchup
Parts:
- PE1: footprint Connector_Wire:SolderWirePad_1x02_P5.08mm_Drill1.5mm -> Connector_Molex:Molex_Mini-Fit_Jr_5566-02A_2x01_P4.20mm_Vertical
- TC1: footprint Connector_Molex:Molex_Mini-Fit_Jr_5566-02A_2x01_P4.20mm_Vertical -> Connector_Wire:SolderWire-2sqmm_1x02_P7.8mm_D2mm_OD3.9mm
Changed lines of the file:
@@
 F 0 "PE1" H 8050 4842 50  0000 C CNN
 F 1 "Peltier_Element" H 8050 4751 50  0000 C CNN
-F 2 "Connector_Wire:SolderWirePad_1x02_P5.08mm_Drill1.5mm" H 8050 4530 50  0001 C CNN
+F 2 "Connector_Molex:Molex_Mini-Fit_Jr_5566-02A_2x01_P4.20mm_Vertical" H 8050 4530 50  0001 C CNN
 F 3 "~" V 8050 4625 50  0001 C CNN
 	1    8050 4600
@@
 F 0 "TC1" V 1527 756 50  0000 R CNN
 F 1 "Thermocouple" V 1618 756 50  0000 R CNN
-F 2 "Connector_Molex:Molex_Mini-Fit_Jr_5566-02A_2x01_P4.20mm_Vertical" H 1025 950 50  0001 C CNN
+F 2 "Connector_Wire:SolderWire-2sqmm_1x02_P7.8mm_D2mm_OD3.9mm" H 1025 950 50  0001 C CNN
 F 3 "~" H 1025 950 50  0001 C CNN
 	1    1600 900
